Commit message: a-a-a

File: robot_desc/urdf/robot.urdf.xacro (robot description, xacro)
@@ -98,4 +98,63 @@
   </collision>
 </link>
+<joint name="camera_joint" type="fixed">
+    <axis xyz="0 1 0" />
+    <origin xyz="0 0 0.4" rpy="0 0 -1.57"/>
+    <parent link="robot_base"/>
+    <child link="camera_link"/>
+  </joint>
+  <!-- Camera -->
+  <link name="camera_link">
+    <collision>
+      <origin xyz="0 0 0" rpy="0 0 0"/>
+      <geometry>
+    <box size="0.1 0.1 0.1"/>
+      </geometry>
+    </collision>
+    <visual>
+      <origin xyz="0 0 0" rpy="0 0 0"/>
+      <geometry>
+    <box size="0.1 0.1 0.1"/>
+      </geometry>
+      <material name="blue"/>
+    </visual>
+    <inertial>
+      <mass value="1e-5" />
+      <origin xyz="0 0 0" rpy="0 0 0"/>
+      <inertia ixx="1e-6" ixy="0" ixz="0" iyy="1e-6" iyz="0" izz="1e-6" />
+    </inertial>
+  </link>
+<!-- camera -->
+  <gazebo reference="camera_link">
+    <sensor type="camera" name="camera1">
+      <update_rate>30.0</update_rate>
+      <camera name="head">
+        <horizontal_fov>1.3962634</horizontal_fov>
+        <image>
+          <width>800</width>
+          <height>800</height>
+          <format>R8G8B8</format>
+        </image>
+        <clip>
+          <near>0.02</near>
+          <far>300</far>
+        </clip>
+      </camera>
+      <plugin name="camera_controller" filename="libgazebo_ros_camera.so">
+        <alwaysOn>true</alwaysOn>
+        <updateRate>0.0</updateRate>
+        <cameraName>rrbot/camera1</cameraName>
+        <imageTopicName>image_raw</imageTopicName>
+        <cameraInfoTopicName>camera_info</cameraInfoTopicName>
+        <frameName>camera_link</frameName>
+        <hackBaseline>0.07</hackBaseline>
+        <distortionK1>0.0</distortionK1>
+        <distortionK2>0.0</distortionK2>
+        <distortionK3>0.0</distortionK3>
+        <distortionT1>0.0</distortionT1>
+        <distortionT2>0.0</distortionT2>
+      </plugin>
+    </sensor>
+  </gazebo>
 <joint name="base_to_lwheel" type="continuous">
   <parent link="robot_base"/>
@@ -113,5 +172,5 @@
   <parent link="robot_base"/>
   <child link="front_holder"/>
-  <origin xyz="0.0 0.8 -0.09" rpy="0 0 0"/>
+  <origin xyz="0.0 -0.8 -0.095" rpy="0 0 0"/>
   <axis xyz="0 0 1"/>
 </joint>
@@ -119,8 +178,8 @@
   <parent link="robot_base"/>
   <child link="back_holder"/>
-  <origin xyz="0.0 -0.8 -0.09" rpy="0 0 0"/>
-  <axis xyz="0 0 1"/>
-</joint>
-<gazebo reference="right_wheel">
+  <origin xyz="0.0 0.8 -0.095" rpy="0 0 0"/>
+  <axis xyz="0 0 1"/>
+</joint>
+<gazebo reference="front_holder">
 <material>Gazebo/Blue</material>
 </gazebo>
@@ -200,5 +259,5 @@
         <scan>
           <horizontal>
-            <samples>720</samples>
+            <samples>100</samples>
             <resolution>1</resolution>
             <min_angle>-1.57</min_angle>
@@ -207,6 +266,6 @@
         </scan>
         <range>
-          <min>0.10</min>
-          <max>30.0</max>
+          <min>0.5</min>
+          <max>5.0</max>
           <resolution>0.01</resolution>
         </range>
